File: hardware_tiny/tiny.kicad_pcb (KiCad board)
At the start: 2 copper layers, 45 x 23 mm, 35 parts, among them P1 USB_OTG, P2 CONN_02X05, P3 CONN_01X05, P4 CONN_01X05, U1 ASM1117-3.3, U2 STM32F103CB, Y1 8M

Commit message: add demo videos
Parts:
- U1: value ASM1117-3.3 -> AMS1117-3.3
Changed lines of the file:
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@@
       (effects (font (size 1 1) (thickness 0.15)))
     )
-    (fp_text value ASM1117-3.3 (at 0 0.762) (layer F.Fab) hide
+    (fp_text value AMS1117-3.3 (at 0 0.762) (layer F.Fab) hide
       (effects (font (size 1 1) (thickness 0.15)))
     )

Commit message: edit
Parts:
- U1: footprint TO_SOT_Packages_SMD:SOT-223 -> footprints:SOT-223
- turned U1 to 270 degrees
- turned U2 to 0 degrees
