File: hardware_tiny/tiny.kicad_pcb (KiCad board)
At the start: 2 copper layers, 45 x 23 mm, 53 parts, among them P1 USB_OTG, P2 CONN_02X05, P3 CONN_01X05, P4 CONN_01X05, U1 AMS1117-3.3, U2 STM32F103CB, Y1 8M

Commit message: edit
Parts:
- P3, P4: footprint Pin_Headers:Pin_Header_Straight_1x05 -> Connector_PinHeader_2.54mm:PinHeader_1x05_P2.54mm_Vertical
