File: hardware_tiny/tiny.sch (KiCad schematic (older format))
At the start: 34 parts, among them P1 USB_OTG, P2 CONN_02X05, P3 CONN_01X05, P4 CONN_01X05, U1 ASM1117-3.3, U2 STM32F103CB, Y1 8M

Commit message: add demo videos
Parts:
- U1: value ASM1117-3.3 -> AMS1117-3.3
Connections:
- wire segments 95 -> 84
Changed lines of the file:
@@
 P 3200 2000
 F 0 "U1" H 3300 1750 50  0000 C CNN
-F 1 "ASM1117-3.3" H 3200 2250 50  0000 C CNN
+F 1 "AMS1117-3.3" H 3200 2250 50  0000 C CNN
 F 2 "TO_SOT_Packages_SMD:SOT-223" H 3200 2000 50  0001 C CNN
 F 3 "" H 3200 2000 50  0000 C CNN
@@
 	3500 2000 3650 2000
 Wire Wire Line
-	1900 2000 2750 2000
-Wire Wire Line
-	2750 2000 2900 2000
+	1900 2000 2900 2000
 Wire Wire Line
 	1900 2100 2450 2100
 Wire Wire Line
-	1900 2200 2100 2200
-Wire Wire Line
-	2100 2200 2300 2200
+	1900 2200 2300 2200
 Connection ~ 3650 2000
 Connection ~ 2750 2000
@@
 	2750 2000 2700 2000
 Wire Wire Line
-	3100 3100 3300 3100
-Wire Wire Line
-	3300 3100 3900 3100
-Wire Wire Line
-	3100 3400 3300 3400
-Wire Wire Line
-	3300 3400 3900 3400
+	3100 3100 3900 3100
+Wire Wire Line
+	3100 3400 3900 3400
 Connection ~ 3300 3100
 Connection ~ 3300 3400
@@
 	4650 2600 5100 2600
 Wire Wire Line
-	6300 5200 6400 5200
-Wire Wire Line
-	6400 5200 6600 5200
-Wire Wire Line
-	6600 5200 6900 5200
+	6300 5200 6900 5200
 Connection ~ 6300 5200
 Connection ~ 6400 5200
@@
 Connection ~ 6600 1800
 Wire Wire Line
-	6300 1800 6400 1800
-Wire Wire Line
-	6400 1800 6600 1800
-Wire Wire Line
-	6600 1800 6900 1800
+	6300 1800 6900 1800
 Wire Wire Line
 	8100 2300 8450 2300
@@
 	1550 3550 1850 3550
 Wire Wire Line
-	1850 3550 1850 3550
-Wire Wire Line
 	1550 3250 1850 3250
-Wire Wire Line
-	1850 3250 1850 3250
-Wire Wire Line
-	1850 3250 1850 3250
 $Comp
 L +3.3V #PWR025
@@
 $EndComp
 $Comp
-L +3.3V #PWR032
+L +3.3V #PWR029
 U 1 1 59842151
 P 9600 1500
-F 0 "#PWR032" H 9600 1350 50  0001 C CNN
+F 0 "#PWR029" H 9600 1350 50  0001 C CNN
 F 1 "+3.3V" H 9600 1640 50  0000 C CNN
 F 2 "" H 9600 1500 50  0000 C CNN

Commit message: edit
Parts:
- added F2: 200mA, Resistor_SMD:R_1210_3225Metric_Pad1.42x2.65mm_HandSolder, symbol tiny-rescue:F_Small
- added LOGO1: MCUSH, logo:mcush_txt_logo, symbol mcush_logo:LOGO
- added TP1: D6, TestPoint:TestPoint_Pad_D1.0mm, symbol Connector:TestPoint
- added TP10: D8, TestPoint:TestPoint_Pad_D1.0mm, symbol Connector:TestPoint
- added TP11: PA15, TestPoint:TestPoint_Pad_D1.0mm, symbol Connector:TestPoint
- added TP12: PB1, TestPoint:TestPoint_Pad_D1.0mm, symbol Connector:TestPoint
- added TP13: PB3, TestPoint:TestPoint_Pad_D1.0mm, symbol Connector:TestPoint
- added TP14: PB4, TestPoint:TestPoint_Pad_D1.0mm, symbol Connector:TestPoint
- added TP15: PB5, TestPoint:TestPoint_Pad_D1.0mm, symbol Connector:TestPoint
- added TP16: PB6, TestPoint:TestPoint_Pad_D1.0mm, symbol Connector:TestPoint
- added TP17: PB7, TestPoint:TestPoint_Pad_D1.0mm, symbol Connector:TestPoint
- added TP2: D7, TestPoint:TestPoint_Pad_D1.0mm, symbol Connector:TestPoint
- added TP3: C13, TestPoint:TestPoint_Pad_D1.0mm, symbol Connector:TestPoint
- added TP4: C14, TestPoint:TestPoint_Pad_D1.0mm, symbol Connector:TestPoint
- added TP5: C15, TestPoint:TestPoint_Pad_D1.0mm, symbol Connector:TestPoint
- added TP6: CS, TestPoint:TestPoint_Pad_D1.0mm, symbol Connector:TestPoint
- added TP7: SCK, TestPoint:TestPoint_Pad_D1.0mm, symbol Connector:TestPoint
- added TP8: MISO, TestPoint:TestPoint_Pad_D1.0mm, symbol Connector:TestPoint
- added TP9: MOSI, TestPoint:TestPoint_Pad_D1.0mm, symbol Connector:TestPoint
- C1, C7: footprint Capacitors_SMD:C_1210_HandSoldering -> Capacitor_SMD:C_1210_3225Metric_Pad1.42x2.65mm_HandSolder; symbol C -> tiny-rescue:C
- C2, C3, C4, C5, C9: footprint Capacitors_SMD:C_0805_HandSoldering -> Capacitor_SMD:C_0805_2012Metric_Pad1.15x1.40mm_HandSolder; symbol C -> tiny-rescue:C
- D1, D2: symbol Led_x2 -> tiny-rescue:Led_x2
- F1: footprint Resistors_SMD:R_1210_HandSoldering -> Resistor_SMD:R_1210_3225Metric_Pad1.42x2.65mm_HandSolder; symbol F_Small -> tiny-rescue:F_Small
- P1: symbol USB_OTG -> tiny-rescue:USB_OTG
- P2: symbol CONN_02X05 -> tiny-rescue:CONN_02X05
- P3, P4: symbol CONN_01X05 -> tiny-rescue:CONN_01X05
- R1, R10, R11, R12, R13, R15, R16, R17, R18, R19, R4, R5, R6, R7, R8, R9: footprint Resistors_SMD:R_0805_HandSoldering -> Resistor_SMD:R_0805_2012Metric_Pad1.15x1.40mm_HandSolder; symbol R -> tiny-rescue:R
- SP1: symbol SPEAKER -> tiny-rescue:SPEAKER
- U1: footprint TO_SOT_Packages_SMD:SOT-223 -> Package_TO_SOT_SMD:SOT-223-3_TabPin2; symbol AP1117D33 -> tiny-rescue:AP1117D33
- U2: footprint footprints:LQFP-48_7x7mm_Pitch0.5mm_HandSoldering -> Package_QFP:LQFP-48_7x7mm_P0.5mm; symbol STM32F103CB -> tiny-rescue:STM32F103CB
- Y1: symbol Crystal -> tiny-rescue:Crystal
Connections:
- net labels added: 3.3V_OUT, C13, C14, C15, D6, D7, D8, PA15, PB1, PB3, PB4, PB5, PB6, PB7
- wire segments 84 -> 115

Commit message: edit
Parts:
- C1, C2, C3, C4, C5, C7, C9: symbol tiny-rescue:C -> tiny-rescue:C-tiny-rescue
- D1, D2: symbol tiny-rescue:Led_x2 -> tiny-rescue:Led_x2-tiny-rescue
- F1, F2: symbol tiny-rescue:F_Small -> tiny-rescue:F_Small-tiny-rescue
- P1: symbol tiny-rescue:USB_OTG -> Connector:USB_B_Mini
- P2: symbol tiny-rescue:CONN_02X05 -> tiny-rescue:CONN_02X05-tiny-rescue
- P3, P4: footprint Pin_Headers:Pin_Header_Straight_1x05 -> Connector_PinHeader_2.54mm:PinHeader_1x05_P2.54mm_Vertical; symbol tiny-rescue:CONN_01X05 -> Connector_Generic:Conn_01x05
- R1, R10, R11, R12, R13, R15, R16, R17, R18, R19, R4, R5, R6, R7, R8, R9: symbol tiny-rescue:R -> tiny-rescue:R-tiny-rescue
- SP1: symbol tiny-rescue:SPEAKER -> tiny-rescue:SPEAKER-tiny-rescue
- U1: symbol tiny-rescue:AP1117D33 -> tiny-rescue:AP1117D33-tiny-rescue
- U2: symbol tiny-rescue:STM32F103CB -> tiny-rescue:STM32F103CB-tiny-rescue
- Y1: symbol tiny-rescue:Crystal -> tiny-rescue:Crystal-tiny-rescue
Connections:
- wire segments 115 -> 114
- no-connect marks 2 -> 1
