File: hardware_tiny_usb_stick/usb_stick.kicad_pcb (KiCad board)
At the start: 2 copper layers, 40 x 15 mm, 27 parts, among them P1 USB_A, P2 CONN_02X05, P4 CONN_01X05, U1 AMS1117-3.3, U2 STM32F103CB, Y1 8M

Commit message: add adc/pwm control
Routing:
- added copper zone on B.Cu, net GND
Changed lines of the file:
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@@
   (general
     (links 79)
-    (no_connects 21)
+    (no_connects 18)
     (area 99.949999 99.949999 140.050001 115.050001)
     (thickness 1.6)
@@
   (via (at 132.6769 105.7021) (size 0.6) (drill 0.4) (layers F.Cu B.Cu) (net 27))
   (segment (start 132.6769 105.7021) (end 132.842 105.8672) (width 0.25) (layer F.Cu) (net 27))
+  (zone (net 2) (net_name GND) (layer B.Cu) (hatch edge 0.508)
+    (connect_pads (clearance 0.508))
+    (min_thickness 0.254)
+    (fill yes (arc_segments 16) (thermal_gap 0.508) (thermal_bridge_width 0.508))
+    (polygon
+      (pts
+        (xy 101.092 126.492) (xy 101.092 141.224) (xy 109.728 141.224) (xy 142.24 141.224) (xy 142.24 125.476)
+        (xy 101.092 125.476) (xy 101.092 126.492)
+      )
+    )
+  )
 )
