File: hardware_tiny_usb_stick/usb_stick.sch (KiCad schematic (older format))
At the start: 27 parts, among them P1 USB_A, P2 CONN_02X05, P4 CONN_01X05, U1 AMS1117-3.3, U2 STM32F103CB, Y1 8M

Commit message: edit
Parts:
- C1, C2, C3, C4, C5, C7, C9: symbol C -> usb_stick-rescue:C
- D1: symbol Led_Small -> usb_stick-rescue:Led_Small
- F1: symbol F_Small -> usb_stick-rescue:F_Small
- P1: symbol USB_A -> usb_stick-rescue:USB_A
- P2: symbol CONN_02X05 -> usb_stick-rescue:CONN_02X05
- P4: symbol CONN_01X05 -> usb_stick-rescue:CONN_01X05
- R1, R10, R11, R12, R13, R17, R18, R4, R5, R7, R8, R9: symbol R -> usb_stick-rescue:R
- U1: symbol AP1117D33 -> usb_stick-rescue:AP1117D33
- U2: symbol STM32F103CB -> usb_stick-rescue:STM32F103CB
- Y1: symbol Crystal -> usb_stick-rescue:Crystal
Connections:
- wire segments 74 -> 82
Changed lines of the file:
@@
-EESchema Schematic File Version 2
-LIBS:power
-LIBS:device
-LIBS:transistors
-LIBS:conn
-LIBS:linear
-LIBS:regul
-LIBS:74xx
-LIBS:cmos4000
-LIBS:adc-dac
-LIBS:memory
-LIBS:xilinx
-LIBS:microcontrollers
-LIBS:dsp
-LIBS:microchip
-LIBS:analog_switches
-LIBS:motorola
-LIBS:texas
-LIBS:intel
-LIBS:audio
-LIBS:interface
-LIBS:digital-audio
-LIBS:philips
-LIBS:display
-LIBS:cypress
-LIBS:siliconi
-LIBS:opto
-LIBS:atmel
-LIBS:contrib
-LIBS:valves
-LIBS:stm32
+EESchema Schematic File Version 4
 LIBS:usb_stick-cache
-EELAYER 25 0
+EELAYER 26 0
 EELAYER END
 $Descr A4 11693 8268
@@
 $EndDescr
 $Comp
-L STM32F103CB U2
+L usb_stick-rescue:STM32F103CB U2
 U 1 1 597ED686
 P 6600 3500
@@
 $EndComp
 $Comp
-L CONN_02X05 P2
+L usb_stick-rescue:CONN_02X05 P2
 U 1 1 597EEA82
 P 9050 4950
@@
 $EndComp
 $Comp
-L C C4
+L usb_stick-rescue:C C4
 U 1 1 597EEC9B
 P 2950 3100
@@
 $EndComp
 $Comp
-L C C5
+L usb_stick-rescue:C C5
 U 1 1 597EECF2
 P 2950 3400
@@
 $EndComp
 $Comp
-L Crystal Y1
+L usb_stick-rescue:Crystal Y1
 U 1 1 597EED5D
 P 3300 3250
@@
 $EndComp
 $Comp
-L F_Small F1
+L usb_stick-rescue:F_Small F1
 U 1 1 597EEDDE
 P 8650 5300
@@
 $EndComp
 $Comp
-L R R7
+L usb_stick-rescue:R R7
 U 1 1 597EF072
 P 4400 1950
@@
 $EndComp
 $Comp
-L AP1117D33 U1
+L usb_stick-rescue:AP1117D33 U1
 U 1 1 597EF5DC
 P 3200 2000
@@
 $EndComp
 $Comp
-L GND #PWR01
+L power:GND #PWR01
 U 1 1 597F4772
 P 2800 3400
@@
 $EndComp
 $Comp
-L GND #PWR02
+L power:GND #PWR02
 U 1 1 597F47A8
 P 2800 3100
@@
 $EndComp
 $Comp
-L C C9
+L usb_stick-rescue:C C9
 U 1 1 597F62F4
 P 4400 2250
@@
 $EndComp
 $Comp
-L GND #PWR03
+L power:GND #PWR03
 U 1 1 597F63AC
 P 4400 2400
@@
 $EndComp
 $Comp
-L +3.3V #PWR04
+L power:+3.3V #PWR04
 U 1 1 597F682B
 P 6300 1800
@@
 $EndComp
 $Comp
-L +3.3V #PWR05
+L power:+3.3V #PWR05
 U 1 1 597F6861
 P 4400 1800
@@
 $EndComp
 $Comp
-L +3.3V #PWR06
+L power:+3.3V #PWR06
 U 1 1 597F68EC
 P 3650 2000
@@
 $EndComp
 $Comp
-L GND #PWR07
+L power:GND #PWR07
 U 1 1 597F6922
 P 3200 2300
@@
 $EndComp
 $Comp
-L +5V #PWR08
+L power:+5V #PWR08
 U 1 1 597F6B30
 P 2750 2000
@@
 $EndComp
 $Comp
-L GND #PWR09
+L power:GND #PWR09
 U 1 1 597F6D0C
 P 1900 2300
@@
 DP
 $Comp
-L C C7
+L usb_stick-rescue:C C7
 U 1 1 597F6FDF
 P 3650 2150
@@
 $EndComp
 $Comp
-L GND #PWR010
+L power:GND #PWR010
 U 1 1 597F70B6
 P 3650 2300
@@
 $EndComp
 $Comp
-L GND #PWR011
+L power:GND #PWR011
 U 1 1 597F73D4
 P 2750 2300
@@
 $EndComp
 $Comp
-L +5V #PWR012
+L power:+5V #PWR012
 U 1 1 597F7482
 P 8550 5300
@@
 OSC_OUT
 $Comp
-L +3.3V #PWR013
+L power:+3.3V #PWR013
 U 1 1 597F9612
 P 5100 2800
@@
 $EndComp
 $Comp
-L GND #PWR014
+L power:GND #PWR014
 U 1 1 597F979B
 P 6300 5200
@@
 $EndComp
 $Comp
-L R R5
+L usb_stick-rescue:R R5
 U 1 1 597FA3C5
 P 3700 4100
@@
 $EndComp
 $Comp
-L GND #PWR015
+L power:GND #PWR015
 U 1 1 597FAE9A
 P 4800 2300
@@
 DP
 $Comp
-L R R4
+L usb_stick-rescue:R R4
 U 1 1 59801AFD
 P 2450 2350
@@
 $EndComp
 $Comp
-L R R1
+L usb_stick-rescue:R R1
 U 1 1 59801D02
 P 2300 2350
@@
 $EndComp
 $Comp
-L R R8
+L usb_stick-rescue:R R8
 U 1 1 59802F35
 P 8950 1800
@@
 $EndComp
 $Comp
-L R R9
+L usb_stick-rescue:R R9
 U 1 1 59803066
 P 8950 1950
@@
 $EndComp
 $Comp
-L R R10
+L usb_stick-rescue:R R10
 U 1 1 598032A0
 P 8950 2100
@@
 $EndComp
 $Comp
-L R R11
+L usb_stick-rescue:R R11
 U 1 1 598035B6
 P 8950 2250
@@
 $EndComp
 $Comp
-L R R12
+L usb_stick-rescue:R R12
 U 1 1 59803827
 P 8950 2400
@@
 $EndComp
 $Comp
-L R R13
+L usb_stick-rescue:R R13
 U 1 1 598038E0
 P 8950 2550
@@
 	3500 2000 3650 2000
 Wire Wire Line
-	1900 2000 2900 2000
+	1900 2000 2750 2000
 Wire Wire Line
 	1900 2100 2450 2100
 Wire Wire Line
-	1900 2200 2300 2200
+	1900 2200 2100 2200
 Connection ~ 3650 2000
 Connection ~ 2750 2000
@@
 	2750 2000 2700 2000
 Wire Wire Line
-	3100 3100 3900 3100
-Wire Wire Line
-	3100 3400 3900 3400
+	3100 3100 3300 3100
+Wire Wire Line
+	3100 3400 3300 3400
 Connection ~ 3300 3100
 Connection ~ 3300 3400
@@
 	4650 2600 5100 2600
 Wire Wire Line
-	6300 5200 6900 5200
+	6300 5200 6400 5200
 Connection ~ 6300 5200
 Connection ~ 6400 5200
@@
 Connection ~ 6600 1800
 Wire Wire Line
-	6300 1800 6900 1800
+	6300 1800 6400 1800
 Wire Wire Line
 	8100 2300 8450 2300
@@
 	8450 4950 8800 4950
 $Comp
-L GND #PWR016
+L power:GND #PWR016
 U 1 1 598044A0
 P 9300 5150
@@
 	9300 5050 9300 5150
 $Comp
-L +3.3V #PWR017
+L power:+3.3V #PWR017
 U 1 1 59804588
 P 8450 5050
@@
 Connection ~ 9300 5150
 $Comp
-L CONN_01X05 P4
+L usb_stick-rescue:CONN_01X05 P4
 U 1 1 598050D5
 P 9400 4050
@@
 $EndComp
 $Comp
-L GND #PWR018
+L power:GND #PWR018
 U 1 1 59805480
 P 9000 4050
@@
 RST
 $Comp
-L +3.3V #PWR019
+L power:+3.3V #PWR019
 U 1 1 59805677
 P 9200 3850
@@
 	4950 3600 5100 3600
 $Comp
-L GND #PWR020
+L power:GND #PWR020
 U 1 1 5981FFFA
 P 4950 3600
@@
 5V_OUT
 $Comp
-L C C2
+L usb_stick-rescue:C C2
 U 1 1 5983C1FA
 P 1550 3400
@@
 $EndComp
 $Comp
-L C C3
+L usb_stick-rescue:C C3
 U 1 1 5983C2A3
 P 1850 3400
@@
 	1550 3250 1850 3250
 $Comp
-L +3.3V #PWR021
+L power:+3.3V #PWR021
 U 1 1 5983C690
 P 1550 3250
@@
 $EndComp
 $Comp
-L GND #PWR022
+L power:GND #PWR022
 U 1 1 5983C6E8
 P 1550 3550
@@
 	2450 2100 2450 2200
 $Comp
-L R R17
+L usb_stick-rescue:R R17
 U 1 1 59816052
 P 2100 2350
@@
 $EndComp
 $Comp
-L +3.3V #PWR023
+L power:+3.3V #PWR023
 U 1 1 5981709A
 P 2100 2500
@@
 Connection ~ 2100 2200
 $Comp
-L GND #PWR024
+L power:GND #PWR024
 U 1 1 598202EF
 P 3350 4100
@@
 	8550 5300 8500 5300
 $Comp
-L R R18
+L usb_stick-rescue:R R18
 U 1 1 59842093
 P 9600 1650
@@
 $EndComp
 $Comp
-L +3.3V #PWR025
+L power:+3.3V #PWR025
 U 1 1 59842151
 P 9600 1500
@@
 3E 24 42 3D 28 80 43 49 0C 1C 4A 62 E0 50 12 03 87 92 18 38 94 C4 C0 A1 24 06 0E 25 31 70 28 89
 81 43 49 0C 1C 4A 62 E0 50 12 03 87 92 18 38 FF 03 DB 50 B2 42 6F C8 55 FC 00 00 00 00 49 45 4E
-44 AE 42 60 82 00
+44 AE 42 60 82
 EndData
 $EndBitmap
@@
 Connection ~ 8800 5150
 $Comp
-L C C1
+L usb_stick-rescue:C C1
 U 1 1 599FC129
 P 2750 2150
@@
 	4800 2300 5100 2300
 $Comp
-L Led_Small D1
+L usb_stick-rescue:Led_Small D1
 U 1 1 5AEC7FF4
 P 3450 4100
@@
 $EndComp
 $Comp
-L USB_A P1
+L usb_stick-rescue:USB_A P1
 U 1 1 5AEC3496
 P 1600 2200
@@
 	0    -1   1    0
 $EndComp
+Wire Wire Line
+	2750 2000 2900 2000
+Wire Wire Line
+	3300 3100 3900 3100
+Wire Wire Line
+	3300 3400 3900 3400
+Wire Wire Line
+	6400 5200 6600 5200
+Wire Wire Line
+	6600 5200 6900 5200
+Wire Wire Line
+	6400 1800 6600 1800
+Wire Wire Line
+	6600 1800 6900 1800
+Wire Wire Line
+	2100 2200 2300 2200
 $EndSCHEMATC
